Commit message: feat: sudah bisa mapping tapi jelek

File: src/ros2_utils/description/omoda.urdf (robot description, URDF)
Before this commit: robot omoda, 7 links, 6 joints
Links:
- added link camera_link
Joints:
- added joint camera_joint: type fixed, parent base_link, child camera_link, origin xyz=0.8 0.0 1.0 rpy=0.0 0.0 0.0

Commit message: feat: aduh lupa

File: src/ros2_utils/description/omoda.urdf (robot description, URDF)
Before this commit: robot omoda, 9 links, 8 joints
Joints:
- joint base_joint: origin xyz=0.0 0.0 1.5 rpy=0.0 0.0 0.0 -> xyz=0.0 0.0 1.60 rpy=0.0 0.0 0.0
- joint lidartengah_joint: origin xyz=0.0 0.0 0.43 rpy=0.0 0.0 0.0 -> xyz=0.0 0.0 0.43 rpy=0.0 0.020 0.0
- joint velodyne1_joint: origin xyz=0.0 -0.45 0.231 rpy=0.78 0.0 0.0 -> xyz=0.0 -0.45 0.231 rpy=0.78 0.008 0.0
- joint velodyne2_joint: origin xyz=0.0 0.45 0.231 rpy=-0.7789 0.0 0.0 -> xyz=0.0 0.45 0.231 rpy=-0.78 0.006 0.0

Commit message: feat: update all ah malas buat commit

File: src/ros2_utils/description/omoda.urdf (robot description, URDF)
Before this commit: robot omoda, 9 links, 8 joints
Links:
- added link gps
Joints:
- added joint gps_joint: type fixed, parent base_lidar, child gps, origin xyz=0.0 0.0 0.43 rpy=0.0 0.0 0.0
